File: kicad/bench-power-supply.sch (KiCad schematic (older format))
At the start: 17 parts

Commit message: Add Propeller code.
Parts:
- removed Q?: BD137, TO-126, symbol BD137
- C3: renamed from C?; value C -> 0.1µ
- Q1: renamed from Q?; value BC547 -> 2N2222
- Q2: renamed from Q?; value BC557 -> 2N4402
- Q3: renamed from Q?; value BD435 -> TIP-120; footprint TO-126 -> TO-220
- R1: renamed from R?; value R -> 10k
- gave numbers to parts that had none: 11
Connections:
- net at Q2.1 (C), R3.1: now also Q3.3 (B)
Other:
- note added: "Current\namplifier"
- note added: "Current\nsense"
- note added: "Voltage from table-top power supply."
- note added: "Voltage\namplifier"
- note added: "Voltage\nfeedback"
- note removed: "5x voltage\namplifier"
- note removed: "Current amplifier"
- note removed: "Current sense"
- note removed: "Voltage feedback"
- moved on the sheet: Q3
Changed lines of the file:
@@
 LIBS:contrib
 LIBS:valves
+LIBS:bench-power-supply-cache
 EELAYER 25 0
 EELAYER END
@@
 $EndDescr
 $Comp
-L BC547 Q?
+L BC547 Q1
 U 1 1 56C76FCC
 P 5900 2000
-F 0 "Q?" H 6100 2075 50  0000 L CNN
-F 1 "BC547" H 6100 2000 50  0000 L CNN
+F 0 "Q1" H 6100 2075 50  0000 L CNN
+F 1 "2N2222" H 6100 2000 50  0000 L CNN
 F 2 "TO-92" H 6100 1925 50  0000 L CIN
 F 3 "" H 5900 2000 50  0000 L CNN
@@
 $EndComp
 $Comp
-L BC557 Q?
+L BC557 Q2
 U 1 1 56C76FE3
 P 6550 1700
-F 0 "Q?" H 6750 1775 50  0000 L CNN
-F 1 "BC557" H 6750 1700 50  0000 L CNN
+F 0 "Q2" H 6750 1775 50  0000 L CNN
+F 1 "2N4402" H 6750 1700 50  0000 L CNN
 F 2 "TO-92" H 6750 1625 50  0000 L CIN
 F 3 "" H 6550 1700 50  0000 L CNN
@@
 $EndComp
 $Comp
-L BD137 Q?
-U 1 1 56C77009
-P 7500 1650
-F 0 "Q?" H 7700 1725 50  0000 L CNN
-F 1 "BD137" H 7700 1650 50  0000 L CNN
-F 2 "TO-126" H 7700 1575 50  0000 L CIN
-F 3 "" H 7500 1650 50  0000 L CNN
-	1    7500 1650
+L BD435 Q3
+U 1 1 56C770DE
+P 7850 1300
+F 0 "Q3" H 8050 1375 50  0000 L CNN
+F 1 "TIP-120" H 8050 1300 50  0000 L CNN
+F 2 "TO-220" H 8050 1225 50  0000 L CIN
+F 3 "" H 7850 1300 50  0000 L CNN
+	1    7850 1300
 	0    -1   -1   0
 $EndComp
 $Comp
-L BD435 Q?
-U 1 1 56C770DE
-P 8250 1300
-F 0 "Q?" H 8450 1375 50  0000 L CNN
-F 1 "BD435" H 8450 1300 50  0000 L CNN
-F 2 "TO-126" H 8450 1225 50  0000 L CIN
-F 3 "" H 8250 1300 50  0000 L CNN
-	1    8250 1300
-	0    -1   -1   0
-$EndComp
-$Comp
-L R R?
+L R R2
 U 1 1 56C7715A
 P 6000 1450
-F 0 "R?" V 6080 1450 50  0000 C CNN
+F 0 "R2" V 6080 1450 50  0000 C CNN
 F 1 "68k" V 6000 1450 50  0000 C CNN
 F 2 "" V 5930 1450 50  0000 C CNN
@@
 $EndComp
 $Comp
-L R R?
+L R R3
 U 1 1 56C77187
 P 6650 2200
-F 0 "R?" V 6730 2200 50  0000 C CNN
+F 0 "R3" V 6730 2200 50  0000 C CNN
 F 1 "4k7" V 6650 2200 50  0000 C CNN
 F 2 "" V 6580 2200 50  0000 C CNN
@@
 $EndComp
 $Comp
-L R R?
+L R R4
 U 1 1 56C771CC
 P 6650 2600
-F 0 "R?" V 6730 2600 50  0000 C CNN
+F 0 "R4" V 6730 2600 50  0000 C CNN
 F 1 "1k" V 6650 2600 50  0000 C CNN
 F 2 "" V 6580 2600 50  0000 C CNN
@@
 $EndComp
 Wire Wire Line
-	6650 2350 6650 2450
+	6650 2350 6650 2400
+Wire Wire Line
+	6650 2400 6650 2450
 Wire Wire Line
 	6000 1200 6000 1300
 Connection ~ 6000 1200
 Wire Wire Line
-	6000 1600 6000 1800
+	6000 1600 6000 1700
+Wire Wire Line
+	6000 1700 6000 1800
 Wire Wire Line
 	6000 2200 6000 2400
@@
 Connection ~ 6650 1200
 Wire Wire Line
-	6650 1950 7500 1950
-Wire Wire Line
-	7500 1950 7500 1850
+	7850 1950 6650 1950
 Connection ~ 6650 1950
-Wire Wire Line
-	7300 1550 7200 1550
-Wire Wire Line
-	7200 1550 7200 1200
 Connection ~ 7200 1200
 Wire Wire Line
-	7700 1550 8250 1550
-Wire Wire Line
-	8250 1550 8250 1500
+	7850 1500 7850 1950
 Wire Wire Line
 	6650 2750 6650 2900
@@
 	6000 1700 6350 1700
 Wire Wire Line
-	6650 1900 6650 2050
+	6650 1900 6650 1950
+Wire Wire Line
+	6650 1950 6650 2050
 Wire Wire Line
 	5400 2000 5700 2000
 $Comp
-L +24V #PWR?
+L +24V #PWR3
 U 1 1 56C77A97
 P 2200 1100
-F 0 "#PWR?" H 2200 950 50  0001 C CNN
+F 0 "#PWR3" H 2200 950 50  0001 C CNN
 F 1 "+24V" H 2200 1240 50  0000 C CNN
 F 2 "" H 2200 1100 50  0000 C CNN
@@
 $EndComp
 $Comp
-L GND #PWR?
+L GND #PWR1
 U 1 1 56C77AEC
 P 1700 6200
-F 0 "#PWR?" H 1700 5950 50  0001 C CNN
+F 0 "#PWR1" H 1700 5950 50  0001 C CNN
 F 1 "GND" H 1700 6050 50  0000 C CNN
 F 2 "" H 1700 6200 50  0000 C CNN
@@
 $EndComp
 $Comp
-L R R?
+L R R5
 U 1 1 56C784C8
 P 9350 1650
-F 0 "R?" V 9430 1650 50  0000 C CNN
+F 0 "R5" V 9430 1650 50  0000 C CNN
 F 1 "47k" V 9350 1650 50  0000 C CNN
 F 2 "" V 9280 1650 50  0000 C CNN
@@
 $EndComp
 $Comp
-L R R?
+L R R6
 U 1 1 56C7851D
 P 9350 2050
-F 0 "R?" V 9430 2050 50  0000 C CNN
+F 0 "R6" V 9430 2050 50  0000 C CNN
 F 1 "10k" V 9350 2050 50  0000 C CNN
 F 2 "" V 9280 2050 50  0000 C CNN
@@
 $EndComp
 $Comp
-L R R?
+L R R7
 U 1 1 56C78552
 P 9350 2750
-F 0 "R?" V 9430 2750 50  0000 C CNN
+F 0 "R7" V 9430 2750 50  0000 C CNN
 F 1 "1Ω" V 9350 2750 50  0000 C CNN
 F 2 "" V 9280 2750 50  0000 C CNN
@@
 Connection ~ 9350 1200
 Wire Wire Line
-	9350 1800 9350 1900
-Wire Wire Line
-	9350 2200 9350 2600
+	9350 1800 9350 1850
+Wire Wire Line
+	9350 1850 9350 1900
+Wire Wire Line
+	9350 2200 9350 2400
+Wire Wire Line
+	9350 2400 9350 2500
+Wire Wire Line
+	9350 2500 9350 2600
 Wire Wire Line
 	9350 2500 8800 2500
@@
 	5750 2750 5750 1300
 Text Notes 5800 2700 0    60   ~ 0
-5x voltage\namplifier
+Voltage\namplifier
 Wire Notes Line
 	5750 1300 7050 1300
@@
 Wire Notes Line
 	8450 750  7150 750
-Text Notes 7200 900  0    60   ~ 0
-Current amplifier
+Text Notes 7200 1000 0    60   ~ 0
+Current\namplifier
 Wire Notes Line
 	9150 1450 9550 1450
@@
 Wire Notes Line
 	9150 3050 9150 2450
-Text Notes 9150 3150 0    60   ~ 0
-Current sense
-Text Notes 9600 1550 0    60   ~ 0
-Voltage feedback
-$Comp
-L ATMEGA328P-P IC?
+Text Notes 9150 3250 0    60   ~ 0
+Current\nsense
+Text Notes 9600 1650 0    60   ~ 0
+Voltage\nfeedback
+$Comp
+L ATMEGA328P-P IC1
 U 1 1 56C79128
 P 4100 3950
-F 0 "IC?" H 3350 5200 50  0000 L BNN
+F 0 "IC1" H 3350 5200 50  0000 L BNN
 F 1 "ATMEGA328P-P" H 4500 2550 50  0000 L BNN
 F 2 "DIL28" H 4100 3950 50  0000 C CIN
@@
 $EndComp
 $Comp
-L LM7805 U?
+L LM7805 U1
 U 1 1 56C79384
 P 2250 1900
-F 0 "U?" H 2400 1704 50  0000 C CNN
+F 0 "U1" H 2400 1704 50  0000 C CNN
 F 1 "LM7805" H 2250 2100 50  0000 C CNN
 F 2 "" H 2250 1900 50  0000 C CNN
@@
 $EndComp
 $Comp
-L C C?
+L C C1
 U 1 1 56C79460
 P 1750 2100
-F 0 "C?" H 1775 2200 50  0000 L CNN
+F 0 "C1" H 1775 2200 50  0000 L CNN
 F 1 ".33µ" H 1775 2000 50  0000 L CNN
 F 2 "" H 1788 1950 50  0000 C CNN
@@
 $EndComp
 $Comp
-L C C?
+L C C2
 U 1 1 56C7949D
 P 2700 2100
-F 0 "C?" H 2725 2200 50  0000 L CNN
+F 0 "C2" H 2725 2200 50  0000 L CNN
 F 1 ".1µ" H 2725 2000 50  0000 L CNN
 F 2 "" H 2738 1950 50  0000 C CNN
@@
 $EndComp
 $Comp
-L BARREL_JACK CON?
+L BARREL_JACK CON1
 U 1 1 56C79582
 P 1100 3400
-F 0 "CON?" H 1100 3650 50  0000 C CNN
+F 0 "CON1" H 1100 3650 50  0000 C CNN
 F 1 "BARREL_JACK" H 1100 3200 50  0000 C CNN
 F 2 "" H 1100 3400 50  0000 C CNN
@@
 $EndComp
 Wire Wire Line
-	1400 6050 9850 6050
+	1400 6050 1700 6050
+Wire Wire Line
+	1700 6050 3100 6050
+Wire Wire Line
+	3100 6050 9850 6050
 Wire Wire Line
 	2200 1100 2200 1200
@@
 Connection ~ 1700 6050
 Wire Wire Line
-	1400 1200 1400 3300
-Wire Wire Line
-	1400 1850 1850 1850
+	1400 1200 1400 1850
+Wire Wire Line
+	1400 1850 1400 3300
+Wire Wire Line
+	1400 1850 1750 1850
+Wire Wire Line
+	1750 1850 1850 1850
 Connection ~ 1400 1850
 Wire Wire Line
@@
 Connection ~ 1750 1850
 Wire Wire Line
-	2650 1850 3100 1850
+	2650 1850 2700 1850
+Wire Wire Line
+	2700 1850 2850 1850
+Wire Wire Line
+	2850 1850 3100 1850
 Wire Wire Line
 	2700 1950 2700 1850
@@
 	1750 2250 1750 2350
 Wire Wire Line
-	1750 2350 2700 2350
+	1750 2350 1900 2350
+Wire Wire Line
+	1900 2350 2250 2350
+Wire Wire Line
+	2250 2350 2700 2350
 Wire Wire Line
 	2700 2350 2700 2250
@@
 Connection ~ 1900 2350
 Wire Wire Line
-	3100 1850 3100 3150
+	3100 1850 3100 2850
+Wire Wire Line
+	3100 2850 3100 3150
 Wire Wire Line
 	3100 2850 3200 2850
@@
 	3200 5050 3100 5050
 Wire Wire Line
-	3100 5050 3100 6050
+	3100 5050 3100 5150
+Wire Wire Line
+	3100 5150 3100 6050
 Connection ~ 3100 6050
 Wire Wire Line
@@
 Connection ~ 3100 5150
 Wire Wire Line
-	6650 2900 9350 2900
-$Comp
-L GND #PWR?
+	6650 2900 7700 2900
+Wire Wire Line
+	7700 2900 9350 2900
+$Comp
+L GND #PWR6
 U 1 1 56C7AF6D
 P 7700 3000
-F 0 "#PWR?" H 7700 2750 50  0001 C CNN
+F 0 "#PWR6" H 7700 2750 50  0001 C CNN
 F 1 "GND" H 7700 2850 50  0000 C CNN
 F 2 "" H 7700 3000 50  0000 C CNN
@@
 	8800 4000 5100 4000
 Wire Wire Line
-	1400 1200 8050 1200
-Wire Wire Line
-	8450 1200 10000 1200
-$Comp
-L GND #PWR?
+	1400 1200 2200 1200
+Wire Wire Line
+	2200 1200 6000 1200
+Wire Wire Line
+	6000 1200 6650 1200
+Wire Wire Line
+	6650 1200 7200 1200
+Wire Wire Line
+	7200 1200 7650 1200
+Wire Wire Line
+	8050 1200 9350 1200
+Wire Wire Line
+	9350 1200 10000 1200
+$Comp
+L GND #PWR2
 U 1 1 56C7B292
 P 1900 2500
-F 0 "#PWR?" H 1900 2250 50  0001 C CNN
+F 0 "#PWR2" H 1900 2250 50  0001 C CNN
 F 1 "GND" H 1900 2350 50  0000 C CNN
 F 2 "" H 1900 2500 50  0000 C CNN
@@
 	1900 2350 1900 2500
 $Comp
-L +5V #PWR?
+L +5V #PWR4
 U 1 1 56C7B3CA
 P 2850 1750
-F 0 "#PWR?" H 2850 1600 50  0001 C CNN
+F 0 "#PWR4" H 2850 1600 50  0001 C CNN
 F 1 "+5V" H 2850 1890 50  0000 C CNN
 F 2 "" H 2850 1750 50  0000 C CNN
@@
 Connection ~ 2850 1850
 $Comp
-L R R?
+L R R1
 U 1 1 56C7B6D5
 P 5450 3150
-F 0 "R?" V 5530 3150 50  0000 C CNN
-F 1 "R" V 5450 3150 50  0000 C CNN
+F 0 "R1" V 5530 3150 50  0000 C CNN
+F 1 "10k" V 5450 3150 50  0000 C CNN
 F 2 "" V 5380 3150 50  0000 C CNN
 F 3 "" H 5450 3150 50  0000 C CNN
@@
 $EndComp
 $Comp
-L C C?
+L C C3
 U 1 1 56C7B72D
 P 5800 3350
-F 0 "C?" H 5825 3450 50  0000 L CNN
-F 1 "C" H 5825 3250 50  0000 L CNN
+F 0 "C3" H 5825 3450 50  0000 L CNN
+F 1 "0.1µ" H 5825 3250 50  0000 L CNN
 F 2 "" H 5838 3200 50  0000 C CNN
 F 3 "" H 5800 3350 50  0000 C CNN
@@
 $EndComp
 $Comp
-L GND #PWR?
+L GND #PWR5
 U 1 1 56C7B7C4
 P 5800 3600
-F 0 "#PWR?" H 5800 3350 50  0001 C CNN
+F 0 "#PWR5" H 5800 3350 50  0001 C CNN
 F 1 "GND" H 5800 3450 50  0000 C CNN
 F 2 "" H 5800 3600 50  0000 C CNN
@@
 	5100 3150 5300 3150
 Wire Wire Line
-	5600 3150 6200 3150
+	5600 3150 5800 3150
+Wire Wire Line
+	5800 3150 6200 3150
 Wire Wire Line
 	5800 3150 5800 3200
@@
 Text Label 10000 1200 0    60   ~ 0
 OUT_POS
+Text Notes 1400 850  0    60   ~ 0
+Voltage from table-top power supply.
 $EndSCHEMATC
